File: Larson SC64anner KiCad Files/Larson SC64anner.kicad_pcb (KiCad board)
At the start: 2 copper layers, 390 x 20 mm, 67 parts, among them J1 Conn_02x03_Counter_Clockwise, J10 Conn_02x03_Counter_Clockwise, J11 Conn_02x03_Counter_Clockwise, J12 Conn_02x03_Counter_Clockwise, J13 Conn_02x03_Counter_Clockwise, J14 Conn_02x03_Counter_Clockwise, J15 Conn_02x03_Counter_Clockwise, J16 Conn_02x03_Counter_Clockwise, J17 Conn_02x03_Counter_Clockwise, J18 Conn_02x03_Counter_Clockwise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

Commit message: no message
Parts:
- added C1: 10uF, Capacitor_THT:CP_Radial_D5.0mm_P2.50mm, F.Cu at (82.0, 32.0)
- added C2: 10uF, Capacitor_THT:CP_Radial_D5.0mm_P2.50mm, F.Cu at (44.0, 32.0)
- added C3: 10uF, Capacitor_THT:CP_Radial_D5.0mm_P2.50mm, F.Cu at (138.9, 33.1)
- added C4: 10nF, Capacitor_THT:C_Disc_D7.5mm_W2.5mm_P5.00mm, F.Cu at (119.6, 36.2)
- added D1: 1N4148, Diode_THT:D_DO-35_SOD27_P7.62mm_Horizontal, F.Cu at (62.1, 34.6)
- added J22: 1xRESET_and_1xEXROM, Connector_PinHeader_2.54mm:PinHeader_1x02_P2.54mm_Vertical, F.Cu at (66.0, 27.0)
- added J23: To Switch, Connector_PinHeader_2.54mm:PinHeader_1x01_P2.54mm_Vertical, F.Cu at (66.0, 34.6)
- added J24: +5V, Connector_PinHeader_2.54mm:PinHeader_1x01_P2.54mm_Vertical, F.Cu at (100.4, 33.9)
- added J25: GND, Connector_PinHeader_2.54mm:PinHeader_1x01_P2.54mm_Vertical, F.Cu at (100.4, 29.9)
- added J26: IRQ, Connector_PinHeader_2.54mm:PinHeader_1x01_P2.54mm_Vertical, F.Cu at (104.5, 23.6)
- added J27: Switch, Connector_PinHeader_2.54mm:PinHeader_1x02_P2.54mm_Vertical, F.Cu at (104.4, 33.9)
- added R26: 10000, Resistor_THT:R_Axial_DIN0207_L6.3mm_D2.5mm_P2.54mm_Vertical, F.Cu at (84.5, 27.0)
- added R27: 10000, Resistor_THT:R_Axial_DIN0207_L6.3mm_D2.5mm_P2.54mm_Vertical, F.Cu at (46.5, 27.0)
- added R28: 150, Resistor_THT:R_Axial_DIN0207_L6.3mm_D2.5mm_P2.54mm_Vertical, F.Cu at (141.2, 26.4)
- added R29: 10k linear, Connector_PinHeader_2.54mm:PinHeader_1x03_P2.54mm_Vertical, F.Cu at (119.6, 33.5)
- added U2: NE555, Package_DIP:DIP-8_W7.62mm, F.Cu at (125.8, 23.1)
- added U3: SN74LVC2G17DBVR_Discontinued, digikey-footprints:SOT-23-6, F.Cu at (100.5, 25.9)
- moved R15 9.75 mm to (136.8, 27.0)
Routing:
- net Net-(C3-Pad2): track 0.00 -> 81.6 mm
- net Net-(J27-Pad2): track 0.00 -> 51.8 mm, vias 0 -> 1
- net Net-(C1-Pad2): track 0.00 -> 45.0 mm
- net Net-(C3-Pad1): track 0.00 -> 36.1 mm
- net Net-(C2-Pad1): track 0.00 -> 34.5 mm
- net Net-(R28-Pad1): track 0.00 -> 30.6 mm
- net Net-(C1-Pad1): track 0.00 -> 30.1 mm
- net Net-(J14-Pad1): track 308.4 -> 338.2 mm
- net Net-(C2-Pad2): track 0.00 -> 27.9 mm
- net Net-(U2-Pad3): track 0.00 -> 21.1 mm, vias 0 -> 1
- net Net-(J12-Pad1): track 335.2 -> 356.3 mm, vias 0 -> 1
- net Net-(J15-Pad2): track 4.26 -> 24.4 mm
- net Net-(J10-Pad1): track 331.9 -> 341.8 mm, vias 2 -> 3
- net Net-(C4-Pad1): track 0.00 -> 7.84 mm
- net Net-(LED15-Pad1): track 2.43 -> 9.44 mm
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Other:
- net class LSC64 added: clearance 0.15, trace_width 0.25, via_dia 0.6, via_drill 0.35
- board text added: "CPU Brake"
- board text added: "Expansionsport-Deluxe-Reset"
- board text added: "Griefed/LSC64"
- board text added: "LSC64"
- board text added: "LSC64 V2.18"
- board text added: "NE555"
- board text added: "by Griefed"
- board text added: "github.com/"
- board text removed: "LSC64 V2.18 - by Griefed - https://github.com/Griefed/LSC64"

Commit message: Add files via upload
Parts:
- removed the J25 at (100.4, 29.9)
- removed J27: Switch, Connector_PinHeader_2.54mm:PinHeader_1x02_P2.54mm_Vertical
- added J26: 1x01, Connector_PinHeader_2.54mm:PinHeader_1x01_P2.54mm_Vertical, F.Cu at (103.2, 24.0)
- J1, J10, J11, J12, J13, J14, J15, J16, J17, J18, J19, J2, J20, J3, J4, J5, J6, J7, J8, J9: value Conn_02x03_Counter_Clockwise -> 2x03
- J21: value Conn_01x02 -> 1x02
- J22: value 1xRESET_and_1xEXROM -> 1x02
- J23: value To Switch -> 1x01
- J24: value +5V -> 1x01
- J25: renamed from J26; value IRQ -> 1x01
- R1, R10, R11, R12, R13, R14, R15, R16, R17, R18, R19, R2, R20, R3, R4, R5, R6, R7, R8, R9: value 80 -> 80 Ohm
- R21, R22, R23, R24, R25: value 10 -> 10 Ohm
- R26, R27: value 10000 -> 10k Ohm
- R28: value 150 -> 150 Ohm
- R29: value 10k linear -> 10k Ohm linear
- U1: value ATtiny85V-10PU -> ATtiny85V-20PU
- U3: value SN74LVC2G17DBVR_Discontinued -> SN74LVC2GU04DCKR
- moved R29 5.08 mm to (124.6, 33.3), turned to 270 degrees
- moved J25 4.86 mm to (99.6, 24.0)
- moved U3 3.60 mm to (102.2, 29.0)
- moved J24 0.20 mm to (100.2, 33.9)
Connections:
- R29 pad 1: Net-(R28-Pad1) -> Net-(J24-Pad1)
- R29 pad 3: Net-(J27-Pad2) -> Net-(R28-Pad1)
- U2 pad 4: Net-(J27-Pad2) -> Net-(J24-Pad1)
- U2 pad 8: Net-(J27-Pad2) -> Net-(J24-Pad1)
- U3 pad 5: Net-(J27-Pad2) -> Net-(J24-Pad1)
Routing:
- net Net-(J27-Pad2): track 51.8 -> 0.00 mm, vias 1 -> 0
- net Net-(J24-Pad1): track 4.00 -> 45.0 mm, vias 0 -> 1
- net Net-(C3-Pad1): track 36.1 -> 58.4 mm
- net Net-(C3-Pad2): track 81.6 -> 74.7 mm
- net Net-(U2-Pad3): track 21.1 -> 22.7 mm
- net Net-(R28-Pad1): track 30.6 -> 29.2 mm
- net Net-(J25-Pad1): track 6.18 -> 5.01 mm
- net Net-(J15-Pad2): track 24.4 -> 23.6 mm

Commit message: Updated PCB
- Touchups
- Added mono / stereo headphone amp circuitry
Parts:
- added C10: 470uF, Capacitor_THT:CP_Radial_D5.0mm_P2.50mm, F.Cu at (255.8, 27.1)
- added C11: 10uF, Capacitor_THT:CP_Radial_D5.0mm_P2.50mm, F.Cu at (271.7, 28.1)
- added C12: 100nF, Capacitor_THT:C_Disc_D7.5mm_W2.5mm_P5.00mm, F.Cu at (237.7, 29.4)
- added C5: 10uF, Capacitor_THT:CP_Radial_D5.0mm_P2.50mm, F.Cu at (157.1, 26.1)
- added C6: 470uF, Capacitor_THT:CP_Radial_D5.0mm_P2.50mm, F.Cu at (157.8, 31.7)
- added C7: 100nF, Capacitor_THT:C_Disc_D7.5mm_W2.5mm_P5.00mm, F.Cu at (175.6, 25.9)
- added C8: 10uF, Capacitor_THT:CP_Radial_D5.0mm_P2.50mm, F.Cu at (204.3, 23.5)
- added C9: 10uF, Capacitor_THT:CP_Radial_D5.0mm_P2.50mm, F.Cu at (252.7, 31.9)
- added J29: 1x01, Connector_PinHeader_2.54mm:PinHeader_1x01_P2.54mm_Vertical, F.Cu at (193.8, 24.0)
- added J30: 1x01, Connector_PinHeader_2.54mm:PinHeader_1x01_P2.54mm_Vertical, F.Cu at (180.6, 26.6)
- added J31: 1x01, Connector_PinHeader_2.54mm:PinHeader_1x01_P2.54mm_Vertical, F.Cu at (197.5, 24.0)
- added J32: 1x01, Connector_PinHeader_2.54mm:PinHeader_1x01_P2.54mm_Vertical, F.Cu at (162.0, 33.0)
- added J33: 1x01, Connector_PinHeader_2.54mm:PinHeader_1x01_P2.54mm_Vertical, F.Cu at (161.5, 28.5)
- added J34: 1x01, Connector_PinHeader_2.54mm:PinHeader_1x01_P2.54mm_Vertical, F.Cu at (180.6, 30.3)
- added J35: 1x01, Connector_PinHeader_2.54mm:PinHeader_1x01_P2.54mm_Vertical, F.Cu at (232.0, 27.6)
- added J36: 1x01, Connector_PinHeader_2.54mm:PinHeader_1x01_P2.54mm_Vertical, F.Cu at (217.4, 23.9)
- added J38: 1x01, Connector_PinHeader_2.54mm:PinHeader_1x01_P2.54mm_Vertical, F.Cu at (237.6, 26.0)
- added J39: 1x01, Connector_PinHeader_2.54mm:PinHeader_1x01_P2.54mm_Vertical, F.Cu at (181.2, 34.3)
- added R30: 18k Ohm, Resistor_THT:R_Axial_DIN0207_L6.3mm_D2.5mm_P2.54mm_Vertical, F.Cu at (159.3, 23.2)
- added R31: 10 Ohm, Resistor_THT:R_Axial_DIN0207_L6.3mm_D2.5mm_P2.54mm_Vertical, F.Cu at (177.7, 34.1)
- added R32: 18k Ohm, Resistor_THT:R_Axial_DIN0207_L6.3mm_D2.5mm_P2.54mm_Vertical, F.Cu at (251.3, 24.8)
- added R33: 10 Ohm, Resistor_THT:R_Axial_DIN0207_L6.3mm_D2.5mm_P2.54mm_Vertical, F.Cu at (220.8, 24.0)
- added U4: LM386N-4_NOPB, digikey-footprints:DIP-8_W7.62mm, F.Cu at (194.1, 27.1)
- added U5: LM386N-4_NOPB, digikey-footprints:DIP-8_W7.62mm, F.Cu at (213.2, 27.1)
- U3: footprint digikey-footprints:SOT-23-6 -> Package_DIP:SMDIP-6_W7.62mm
- moved J26 38.3 mm to (141.5, 22.9)
- moved R10 12.6 mm to (233.3, 32.3)
- moved J24 12.2 mm to (105.5, 22.9)
- moved R11 9.32 mm to (211.9, 24.0), turned to 0 degrees
- moved J25 2.17 mm to (101.5, 22.9)
- moved U3 1.29 mm to (102.3, 30.3), turned to 270 degrees
- moved R12 0.48 mm to (184.0, 26.3)
Connections:
- J2 pad 1: Net-(J2-Pad1) -> Net-(J11-Pad1)
- J2 pad 3: Net-(J2-Pad1) -> Net-(J11-Pad1)
- J2 pad 5: Net-(J2-Pad1) -> Net-(J11-Pad1)
Routing:
- net Net-(C11-Pad2): track 0.00 -> 138.2 mm, vias 0 -> 2
- net Net-(C6-Pad1): track 0.00 -> 62.9 mm, vias 0 -> 2
- net Net-(C11-Pad1): track 0.00 -> 60.3 mm, vias 0 -> 2
- net Net-(J11-Pad1): track 296.4 -> 352.6 mm, vias 2 -> 4
- net Net-(C10-Pad1): track 0.00 -> 50.4 mm
- net Net-(R32-Pad1): track 0.00 -> 39.7 mm, vias 0 -> 1
- net Net-(R30-Pad1): track 0.00 -> 36.7 mm
- net Net-(C5-Pad2): track 0.00 -> 35.1 mm
- net Net-(J12-Pad1): track 356.3 -> 387.9 mm, vias 1 -> 2
- net Net-(C10-Pad2): track 0.00 -> 27.9 mm
- net Net-(C12-Pad2): track 0.00 -> 21.8 mm, vias 0 -> 1
- net Net-(J35-Pad1): track 0.00 -> 17.7 mm
- net Net-(J14-Pad1): track 338.2 -> 353.3 mm
- net Net-(J10-Pad1): track 341.8 -> 355.7 mm
- net Net-(C3-Pad1): track 58.4 -> 45.0 mm
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Other:
- board text added: "Mono & Stereo Headphone Amp"
