File: Larson SC64anner KiCad Files/Larson SC64anner.kicad_pcb (KiCad board)
At the start: 2 copper layers, 390 x 20 mm, 104 parts, among them J1 2x03, J10 2x03, J11 2x03, J12 2x03, J13 2x03, J14 2x03, J15 2x03, J16 2x03, J17 2x03, J18 2x03, J19 2x03, J2 2x03, J20 2x03, J21 1x02, J22 1x01, J23 1x01, J24 1x01, J25 1x01, J26 2x05, J27 1x01, J29 1x01, J3 2x03, J31 1x01, J32 1x01, J35 1x01, J36 1x01, J38 1x01, J4 2x03, J5 2x03, J6 2x03, J7 2x03, J8 2x03, J9 2x03, U1 ATtiny85V-20PU, U2 NE555, U3 SN74LVC2GU04DCKR, U4 LM386N-4_NOPB, U5 LM386N-4_NOPB

Commit message: Various
-Added a sociel preview with the LED part of the schematic in the background
-Filled the unsued zones of the pcb with copper fields, to increase production quality due to equal spread of copper layers (galvanic index)
Routing:
- net Net-(C11-Pad2): track 381.0 -> 416.3 mm
- added copper zone on B.Cu, net (none)
- added copper zone on F.Cu, net (none)
- removed copper zone on F.Cu, net Net-(C11-Pad2)
Other:
- board text removed: "Griefed/LSC64"
- board text removed: "by Griefed"
- board text removed: "github.com/"
Changed lines of the file:
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@@
   (general
     (thickness 1.6)
-    (drawings 156)
-    (tracks 1014)
+    (drawings 153)
+    (tracks 1028)
     (zones 0)
     (modules 104)
@@
     (descr "Through hole straight pin header, 1x01, 2.54mm pitch, single row")
     (tags "Through hole pin header THT 1x01 2.54mm single row")
-    (fp_text reference J24 (at 0 -2.33) (layer F.SilkS)
+    (fp_text reference J24 (at -2.05 0.4 90) (layer F.SilkS)
       (effects (font (size 1 1) (thickness 0.15)))
     )
@@
     (descr "Resistor, Axial_DIN0207 series, Axial, Vertical, pin pitch=2.54mm, 0.25W = 1/4W, length*diameter=6.3*2.5mm^2, http://cdn-reichelt.de/documents/datenblatt/B400/1_4W%23YAG.pdf")
     (tags "Resistor Axial_DIN0207 series Axial Vertical pin pitch 2.54mm 0.25W = 1/4W length 6.3mm diameter 2.5mm")
-    (fp_text reference R13 (at -2.46 0 180) (layer F.SilkS)
+    (fp_text reference R13 (at 4.45 0 180) (layer F.SilkS)
       (effects (font (size 1 1) (thickness 0.15)))
     )
@@
     (descr "Resistor, Axial_DIN0207 series, Axial, Vertical, pin pitch=2.54mm, 0.25W = 1/4W, length*diameter=6.3*2.5mm^2, http://cdn-reichelt.de/documents/datenblatt/B400/1_4W%23YAG.pdf")
     (tags "Resistor Axial_DIN0207 series Axial Vertical pin pitch 2.54mm 0.25W = 1/4W length 6.3mm diameter 2.5mm")
-    (fp_text reference R15 (at -2.46 0 180) (layer F.SilkS)
+    (fp_text reference R15 (at -2.1 0.85 180) (layer F.SilkS)
       (effects (font (size 1 1) (thickness 0.15)))
     )
@@
     (descr "Resistor, Axial_DIN0207 series, Axial, Vertical, pin pitch=2.54mm, 0.25W = 1/4W, length*diameter=6.3*2.5mm^2, http://cdn-reichelt.de/documents/datenblatt/B400/1_4W%23YAG.pdf")
     (tags "Resistor Axial_DIN0207 series Axial Vertical pin pitch 2.54mm 0.25W = 1/4W length 6.3mm diameter 2.5mm")
-    (fp_text reference R16 (at -2.46 0 180) (layer F.SilkS)
+    (fp_text reference R16 (at -1.96 -1.3 180) (layer F.SilkS)
       (effects (font (size 1 1) (thickness 0.15)))
     )
@@
     (descr "Resistor, Axial_DIN0207 series, Axial, Vertical, pin pitch=2.54mm, 0.25W = 1/4W, length*diameter=6.3*2.5mm^2, http://cdn-reichelt.de/documents/datenblatt/B400/1_4W%23YAG.pdf")
     (tags "Resistor Axial_DIN0207 series Axial Vertical pin pitch 2.54mm 0.25W = 1/4W length 6.3mm diameter 2.5mm")
-    (fp_text reference R21 (at -2.46 0 -90) (layer F.SilkS)
+    (fp_text reference R21 (at -2.46 0 90) (layer F.SilkS)
       (effects (font (size 1 1) (thickness 0.15)))
     )
@@
     (descr "Resistor, Axial_DIN0207 series, Axial, Vertical, pin pitch=2.54mm, 0.25W = 1/4W, length*diameter=6.3*2.5mm^2, http://cdn-reichelt.de/documents/datenblatt/B400/1_4W%23YAG.pdf")
     (tags "Resistor Axial_DIN0207 series Axial Vertical pin pitch 2.54mm 0.25W = 1/4W length 6.3mm diameter 2.5mm")
-    (fp_text reference R22 (at -2.46 0 -90) (layer F.SilkS)
+    (fp_text reference R22 (at -2.16 0 90) (layer F.SilkS)
       (effects (font (size 1 1) (thickness 0.15)))
     )
@@
     (descr "Resistor, Axial_DIN0207 series, Axial, Vertical, pin pitch=2.54mm, 0.25W = 1/4W, length*diameter=6.3*2.5mm^2, http://cdn-reichelt.de/documents/datenblatt/B400/1_4W%23YAG.pdf")
     (tags "Resistor Axial_DIN0207 series Axial Vertical pin pitch 2.54mm 0.25W = 1/4W length 6.3mm diameter 2.5mm")
-    (fp_text reference R23 (at -2.46 0 270) (layer F.SilkS)
+    (fp_text reference R23 (at 4.3 0 270) (layer F.SilkS)
       (effects (font (size 1 1) (thickness 0.15)))
     )
@@
     (descr "Resistor, Axial_DIN0207 series, Axial, Vertical, pin pitch=2.54mm, 0.25W = 1/4W, length*diameter=6.3*2.5mm^2, http://cdn-reichelt.de/documents/datenblatt/B400/1_4W%23YAG.pdf")
     (tags "Resistor Axial_DIN0207 series Axial Vertical pin pitch 2.54mm 0.25W = 1/4W length 6.3mm diameter 2.5mm")
-    (fp_text reference R26 (at -2.46 0 270) (layer F.SilkS)
+    (fp_text reference R26 (at 1.24 2.2) (layer F.SilkS)
       (effects (font (size 1 1) (thickness 0.15)))
     )
@@
   (gr_line (start 349.2 34.6) (end 349.2 28.9) (layer F.SilkS) (width 0.3))
   (gr_line (start 346.4 33.8) (end 352 33.8) (layer F.SilkS) (width 0.12))
-  (gr_text Griefed/LSC64 (at 383.9 30.3 270) (layer F.SilkS)
-    (effects (font (size 1.5 1.5) (thickness 0.3)))
-  )
-  (gr_text github.com/ (at 386.3 30.3 270) (layer F.SilkS)
-    (effects (font (size 1.5 1.5) (thickness 0.3)))
-  )
-  (gr_text "by Griefed" (at 388.7 30 270) (layer F.SilkS)
-    (effects (font (size 1.5 1.5) (thickness 0.3)))
-  )
-  (gr_text "LSC64 V2.18" (at 390.6 30.3 270) (layer F.SilkS)
+  (gr_text "LSC64 V2.18" (at 349.2 38) (layer F.SilkS)
     (effects (font (size 1.5 1.5) (thickness 0.3)))
   )
@@
   (segment (start 260.75 25.2) (end 260.75 25.05) (width 0.25) (layer F.Cu) (net 107))
   (segment (start 260.75 25.05) (end 261.6 24.2) (width 0.25) (layer F.Cu) (net 107))
-  (segment (start 261.6 24.2) (end 272.4 24.2) (width 0.25) (layer F.Cu) (net 107))
-  (segment (start 416.05 34.3) (end 415 34.3) (width 0.25) (layer F.Cu) (net 107))
-  (segment (start 276.4 22.3) (end 277 21.7) (width 0.25) (layer F.Cu) (net 107))
-  (segment (start 277 21.7) (end 416.15 21.7) (width 0.25) (layer F.Cu) (net 107))
-  (segment (start 416.15 21.7) (end 416.7 22.25) (width 0.25) (layer F.Cu) (net 107))
-  (segment (start 416.7 22.25) (end 416.7 33.65) (width 0.25) (layer F.Cu) (net 107))
-  (segment (start 416.7 33.65) (end 416.05 34.3) (width 0.25) (layer F.Cu) (net 107))
   (segment (start 178.56863 22.5) (end 177.7 23.36863) (width 0.25) (layer F.Cu) (net 107))
   (segment (start 177.7 23.36863) (end 177.7 24.5) (width 0.25) (layer F.Cu) (net 107))
   (segment (start 232.6 22.5) (end 178.56863 22.5) (width 0.25) (layer F.Cu) (net 107))
   (segment (start 234.5 24.4) (end 232.6 22.5) (width 0.25) (layer F.Cu) (net 107))
+  (segment (start 262.36 23.44) (end 272.86 23.44) (width 0.25) (layer F.Cu) (net 107))
+  (segment (start 261.6 24.2) (end 262.36 23.44) (width 0.25) (layer F.Cu) (net 107))
+  (segment (start 277.14 21.7) (end 275.4 23.44) (width 0.25) (layer F.Cu) (net 107))
+  (segment (start 415 34.3) (end 416.05 34.3) (width 0.25) (layer F.Cu) (net 107))
+  (segment (start 416.7 22.25) (end 416.15 21.7) (width 0.25) (layer F.Cu) (net 107))
+  (segment (start 416.05 34.3) (end 416.7 33.65) (width 0.25) (layer F.Cu) (net 107))
+  (segment (start 416.7 33.65) (end 416.7 22.25) (width 0.25) (layer F.Cu) (net 107))
+  (segment (start 416.15 21.7) (end 277.14 21.7) (width 0.25) (layer F.Cu) (net 107))
+  (segment (start 272.86 33.6) (end 272.86 31.06) (width 0.6) (layer F.Cu) (net 107))
+  (segment (start 272.86 31.06) (end 272.86 28.52) (width 0.6) (layer F.Cu) (net 107))
+  (segment (start 272.86 28.52) (end 272.86 25.98) (width 0.6) (layer F.Cu) (net 107))
+  (segment (start 272.86 25.98) (end 272.86 23.44) (width 0.6) (layer F.Cu) (net 107))
+  (segment (start 275.4 33.6) (end 275.4 31.06) (width 0.6) (layer F.Cu) (net 107))
+  (segment (start 275.4 31.06) (end 275.4 28.52) (width 0.6) (layer F.Cu) (net 107))
+  (segment (start 275.4 28.52) (end 275.4 25.98) (width 0.6) (layer F.Cu) (net 107))
+  (segment (start 275.4 25.98) (end 275.4 23.44) (width 0.6) (layer F.Cu) (net 107))
+  (segment (start 272.86 23.44) (end 275.4 23.44) (width 0.6) (layer F.Cu) (net 107))
+  (segment (start 275.4 33.6) (end 272.86 33.6) (width 0.6) (layer F.Cu) (net 107))
+  (segment (start 272.86 31.06) (end 275.4 31.06) (width 0.6) (layer F.Cu) (net 107))
+  (segment (start 275.4 28.52) (end 272.86 28.52) (width 0.6) (layer F.Cu) (net 107))
+  (segment (start 272.86 25.98) (end 275.4 25.98) (width 0.6) (layer F.Cu) (net 107))
   (via (at 230.95 24.25) (size 0.6) (drill 0.35) (layers F.Cu B.Cu) (net 108))
   (segment (start 254.3 26) (end 254.4 25.9) (width 0.25) (layer B.Cu) (net 108))
@@
   (segment (start 413.787919 23.3) (end 412.45 23.3) (width 0.25) (layer F.Cu) (net 119))
   (segment (start 414.99 23.3) (end 413.787919 23.3) (width 0.25) (layer F.Cu) (net 119))
-  (zone (net 107) (net_name "Net-(C11-Pad2)") (layer F.Cu) (hatch edge 0.508)
-    (connect_pads yes (clearance 0.508))
+  (zone (net 0) (net_name "") (layer F.Cu) (hatch edge 0.508)
+    (connect_pads (clearance 0.508))
+    (min_thickness 0.254)
+    (fill yes (arc_segments 32) (thermal_gap 0.508) (thermal_bridge_width 0.508))
+    (polygon
+      (pts
+        (xy 419 40) (xy 29 40) (xy 29 20) (xy 419 20)
+      )
+    )
+  )
+  (zone (net 0) (net_name "") (layer B.Cu) (hatch edge 0.508)
+    (connect_pads (clearance 0.508))
     (min_thickness 0.254)
     (fill yes (arc_segments 32) (thermal_gap 0.508) (thermal_bridge_width 0.508))
     (polygon
       (pts
-        (xy 276.6 35) (xy 271.6 35) (xy 271.6 22.1) (xy 276.6 22.1)
+        (xy 419 40) (xy 29 40) (xy 29 20) (xy 419 20)
       )
     )

Commit message: Updated PCB
-Cleaned up the silklayer which resulted in redoing screenshots and gerber files etc.
Other:
- board text added: "https://github.com/Griefed/LSC64"
- board text removed: "LSC64 V2.18"

Commit message: Minor touchups
Routing:
- net Net-(J1-Pad1): track 186.0 -> 187.0 mm
- net Net-(C11-Pad2): vias 5 -> 4
Other:
- net class LSC64: clearance 0.15 -> 0.2

Commit message: More cleanups
Cleaned the PCB up some more.
Parts:
- moved C3 1.20 mm to (140.0, 33.5)
Routing:
- net Net-(J35-Pad1): track 38.7 -> 30.7 mm
- net Net-(C11-Pad2): track 416.3 -> 419.3 mm, vias 4 -> 3
- net Net-(C10-Pad1): track 39.4 -> 36.5 mm
- net Net-(J36-Pad1): track 32.3 -> 29.6 mm
- net Net-(R32-Pad1): track 35.1 -> 37.5 mm
- net Net-(J14-Pad1): track 357.9 -> 359.7 mm, vias 2 -> 0
- net Net-(C3-Pad2): track 75.3 -> 76.7 mm
- net Net-(C10-Pad2): track 53.7 -> 53.3 mm, vias 2 -> 1
- removed copper zone on B.Cu, net (none)
- removed copper zone on F.Cu, net (none)
Other:
- net class Default: clearance 0.15 -> 0.2; trace_width 0.6 -> 0.25; via_drill 0.4 -> 0.35
- net class LSC64: via_dia 0.6 -> 0.8
- rule trace_clearance: 0.15 -> 0.2
